File: hardware/EAGLE/badge.brd (EAGLE design)
At the start: 47 x 47 mm, 9 parts, among them SW1 SWITCH, X1 BATTERYHOLDER_SMD

Commit message: changed resistor to correct value
Parts:
- R1, R2, R3: value 4.7 -> 100R
Changed lines of the file:
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@@
 <?xml version="1.0" encoding="utf-8"?>
 <!DOCTYPE eagle SYSTEM "eagle.dtd">
-<eagle version="9.2.0">
+<eagle version="9.5.0">
 <drawing>
 <settings>
@@
 </autorouter>
 <elements>
-<element name="SW1" library="badge" package="SWITCH" value="SWITCH" x="23.4958" y="40.506">
+<element name="SW1" library="badge" package="SWITCH" value="SWITCH" x="23.4958" y="40.506" smashed="yes">
 <attribute name="NAME" x="19.2783" y="42.926" size="1.27" layer="25" font="vector" ratio="20"/>
 </element>
-<element name="X1" library="badge" package="BATTERYHOLDER_SMD" value="BATTERYHOLDER_SMD" x="23.4958" y="20.506" rot="MR180"/>
-<element name="R1" library="badge" package="0207/10" value="4.7" x="23.4958" y="8.506">
+<element name="X1" library="badge" package="BATTERYHOLDER_SMD" value="BATTERYHOLDER_SMD" x="23.4958" y="20.506" smashed="yes" rot="MR180"/>
+<element name="R1" library="badge" package="0207/10" value="100R" x="23.4958" y="8.506" smashed="yes">
 <attribute name="NAME" x="18.6958" y="7.506" size="1.27" layer="25" font="vector" ratio="20" rot="R270"/>
 </element>
-<element name="R2" library="badge" package="0207/10" value="4.7" x="34.6558" y="38.806" rot="R323">
+<element name="R2" library="badge" package="0207/10" value="100R" x="34.6558" y="38.806" smashed="yes" rot="R323">
 <attribute name="NAME" x="32.9376375" y="38.315659375" size="1.27" layer="25" font="vector" ratio="20" rot="R323" align="top-left"/>
 </element>
-<element name="R3" library="badge" package="0207/10" value="4.7" x="12.3358" y="38.806" rot="R217">
+<element name="R3" library="badge" package="0207/10" value="100R" x="12.3358" y="38.806" smashed="yes" rot="R217">
 <attribute name="NAME" x="14.34679375" y="38.526009375" size="1.27" layer="25" font="vector" ratio="20" rot="R217"/>
 </element>
-<element name="LED1" library="badge" package="LED5MM" value="LED" x="23.4958" y="4.006" rot="R270">
+<element name="LED1" library="badge" package="LED5MM" value="LED" x="23.4958" y="4.006" smashed="yes" rot="R270">
 <attribute name="NAME" x="27.2958" y="6.806" size="1.27" layer="25" font="vector" ratio="20" rot="R270"/>
 </element>
-<element name="LED2" library="badge" package="LED5MM" value="LED" x="40.9958" y="31.006" rot="R270">
+<element name="LED2" library="badge" package="LED5MM" value="LED" x="40.9958" y="31.006" smashed="yes" rot="R270">
 <attribute name="NAME" x="38.7958" y="26.706" size="1.27" layer="25" font="vector" ratio="20"/>
 </element>
-<element name="LED3" library="badge" package="LED5MM" value="LED" x="5.9958" y="31.006" rot="R270">
+<element name="LED3" library="badge" package="LED5MM" value="LED" x="5.9958" y="31.006" smashed="yes" rot="R270">
 <attribute name="NAME" x="3.7958" y="26.706" size="1.27" layer="25" font="vector" ratio="20"/>
 </element>
-<element name="NEEDLE" library="badge" package="NEEDLE_PAD" value="NEEDLE" x="23.4958" y="34.506" rot="MR0"/>
+<element name="NEEDLE" library="badge" package="NEEDLE_PAD" value="NEEDLE" x="23.4958" y="34.506" smashed="yes" rot="MR0"/>
 </elements>
 <signals>
